Commit message: fixed urdf model

File: jackal_description/urdf/jackal_all.urdf.xacro (robot description, xacro)
@@ -251,5 +251,5 @@
   </joint>
   <!-- Adding lidar frame -->
-  <!-- <link name="os1_sensor">
+  <link name="lidar_mounting_frame">
 	<origin rpy="0 0 0" xyz="0 0 0"/>
 	<visual>
@@ -288,10 +288,4 @@
       		<material name="white"/>
     	</visual>
-	<visual>
-      		<origin rpy="0 0 1.5707" xyz="0 0 0.0365"/>
-      		<geometry>
-        		<mesh filename="package://jackal_description/meshes/os1_64.dae"/>
-      		</geometry>
-    	</visual>
 	 <collision>
       		<origin xyz="0 0 0"/>
@@ -300,17 +294,14 @@
       		</geometry>
     	</collision>
-  </link> -->
-  <link name="lidar_mount_link">
-    <origin xyz="0 0 0" rpy="0 0 0"/>
   </link>
   <joint name="lidar_mount_joint" type="fixed">
 	    <parent link="enclosure_mount_link"/>
-    	<child link="lidar_mount_link"/>
+    	<child link="lidar_mounting_frame"/>
 	<!--x = 0.0065 + 0.06, z= 0.07 + 0.07 + 0.005-->
       <origin xyz="0.0665 0 0.145"/>
   </joint>
   <xacro:include filename="$(find jackal_description)/urdf/OS1-64.urdf.xacro"/>
-  <OS1-64 parent="lidar_mount_link" name="os1-64">
-    <origin xyz="0 0 0.00" rpy="0 0 0" />
+  <OS1-64 parent="lidar_mounting_frame" name="os1-64">
+    <origin xyz="0 0 0.035" rpy="0 0 0" />
   </OS1-64>
   <!-- Bring in simulation data for Gazebo. -->

Commit message: rearranged ouster plugin folder, minor fixes in jackal xacro file

File: jackal_description/urdf/jackal_all.urdf.xacro (robot description, xacro)
@@ -258,5 +258,5 @@
         		<box size="0.14 0.14 0.005"/>
       		</geometry>
-      		<material name="white"/>
+          <material name="dark_grey" />
     	</visual>
 	<visual>
@@ -265,5 +265,5 @@
         		<cylinder length="0.07" radius="0.005"/>
       		</geometry>
-      		<material name="white"/>
+          <material name="dark_grey" />
     	</visual>
    	<visual>
@@ -272,5 +272,5 @@
         		<cylinder length="0.07" radius="0.005"/>
       		</geometry>
-      		<material name="white"/>
+          <material name="dark_grey" />
     	</visual>
 	<visual>
@@ -279,5 +279,5 @@
         		<cylinder length="0.07" radius="0.005"/>
       		</geometry>
-      		<material name="white"/>
+          <material name="dark_grey" />
     	</visual>
 	<visual>
@@ -286,5 +286,5 @@
         		<cylinder length="0.07" radius="0.005"/>
       		</geometry>
-      		<material name="white"/>
+          <material name="dark_grey" />
     	</visual>
 	 <collision>

Commit message: config to make ouster optional

File: jackal_description/urdf/jackal_all.urdf.xacro (robot description, xacro)
@@ -306,59 +306,61 @@
     </sensor>
   </gazebo>
-  <!-- Adding lidar frame -->
-  <link name="lidar_mounting_frame">
-	<origin rpy="0 0 0" xyz="0 0 0"/>
-	<visual>
-      		<origin rpy="0 0 0" xyz="0 0 -0.0025"/>
-      		<geometry>
-        		<box size="0.14 0.14 0.005"/>
-      		</geometry>
-          <material name="dark_grey" />
-    	</visual>
-	<visual>
-      		<origin rpy="0 0 0" xyz="0.06 0.06 -0.04"/>
-      		<geometry>
-        		<cylinder length="0.07" radius="0.005"/>
-      		</geometry>
-          <material name="dark_grey" />
-    	</visual>
-   	<visual>
-      		<origin rpy="0 0 0" xyz="-0.06 0.06 -0.04"/>
-      		<geometry>
-        		<cylinder length="0.07" radius="0.005"/>
-      		</geometry>
-          <material name="dark_grey" />
-    	</visual>
-	<visual>
-      		<origin rpy="0 0 0" xyz="0.06 -0.06 -0.04"/>
-      		<geometry>
-        		<cylinder length="0.07" radius="0.005"/>
-      		</geometry>
-          <material name="dark_grey" />
-    	</visual>
-	<visual>
-      		<origin rpy="0 0 0" xyz="-0.06 -0.06 -0.04"/>
-      		<geometry>
-        		<cylinder length="0.07" radius="0.005"/>
-      		</geometry>
-          <material name="dark_grey" />
-    	</visual>
-	 <collision>
-      		<origin xyz="0 0 0"/>
-      		<geometry>
-        		<box size="0.14 0.14 0.16"/>
-      		</geometry>
-    	</collision>
-  </link>
-  <joint name="lidar_mount_joint" type="fixed">
-	    <parent link="enclosure_mount_link"/>
-    	<child link="lidar_mounting_frame"/>
-	<!--x = 0.0065 + 0.06, z= 0.07 + 0.07 + 0.005-->
-      <origin xyz="0.0665 0 0.145"/>
-  </joint>
-  <xacro:include filename="$(find jackal_description)/urdf/OS1-64.urdf.xacro"/>
-  <xacro:OS1-64 parent="lidar_mounting_frame" name="os1-64">
-    <origin xyz="0 0 0.035" rpy="0 0 0" />
-  </xacro:OS1-64>
+  <xacro:if value="$(optenv OUSTER 0)">
+    <!-- Adding lidar frame -->
+    <link name="lidar_mounting_frame">
+    <origin rpy="0 0 0" xyz="0 0 0"/>
+    <visual>
+            <origin rpy="0 0 0" xyz="0 0 -0.0025"/>
+            <geometry>
+              <box size="0.14 0.14 0.005"/>
+            </geometry>
+            <material name="dark_grey" />
+        </visual>
+    <visual>
+            <origin rpy="0 0 0" xyz="0.06 0.06 -0.04"/>
+            <geometry>
+              <cylinder length="0.07" radius="0.005"/>
+            </geometry>
+            <material name="dark_grey" />
+        </visual>
+      <visual>
+            <origin rpy="0 0 0" xyz="-0.06 0.06 -0.04"/>
+            <geometry>
+              <cylinder length="0.07" radius="0.005"/>
+            </geometry>
+            <material name="dark_grey" />
+        </visual>
+    <visual>
+            <origin rpy="0 0 0" xyz="0.06 -0.06 -0.04"/>
+            <geometry>
+              <cylinder length="0.07" radius="0.005"/>
+            </geometry>
+            <material name="dark_grey" />
+        </visual>
+    <visual>
+            <origin rpy="0 0 0" xyz="-0.06 -0.06 -0.04"/>
+            <geometry>
+              <cylinder length="0.07" radius="0.005"/>
+            </geometry>
+            <material name="dark_grey" />
+        </visual>
+    <collision>
+            <origin xyz="0 0 0"/>
+            <geometry>
+              <box size="0.14 0.14 0.16"/>
+            </geometry>
+        </collision>
+    </link>
+    <joint name="lidar_mount_joint" type="fixed">
+        <parent link="enclosure_mount_link"/>
+        <child link="lidar_mounting_frame"/>
+    <!--x = 0.0065 + 0.06, z= 0.07 + 0.07 + 0.005-->
+        <origin xyz="0.0665 0 0.145"/>
+    </joint>
+    <xacro:include filename="$(find jackal_description)/urdf/OS1-64.urdf.xacro"/>
+    <xacro:OS1-64 parent="lidar_mounting_frame" name="os1-64">
+      <origin xyz="0 0 0.035" rpy="0 0 0" />
+    </xacro:OS1-64>
+  </xacro:if>
   <!-- Bring in simulation data for Gazebo. -->
   <xacro:include filename="$(find jackal_description)/urdf/jackal.gazebo" />
